File: kicad/LoadMouth.kicad_pcb (KiCad board)
At the start: 2 copper layers, 0 parts

Commit message: Started layout
Parts:
- added C1: C, Capacitors_SMD:C_1210_HandSoldering, F.Cu at (161.3, 85.1)
- added C2: C, Capacitors_SMD:C_1210_HandSoldering, F.Cu at (176.5, 97.8)
- added C3: C, Capacitors_SMD:C_1210_HandSoldering, F.Cu at (188.0, 78.7)
- added C4: C, Capacitors_SMD:C_1210_HandSoldering, F.Cu at (182.9, 87.6)
- added P1: CONN_01X02, Pin_Headers:Pin_Header_Straight_1x02, F.Cu at (154.9, 85.1)
- added P2: CONN_01X02, Pin_Headers:Pin_Header_Straight_1x02, F.Cu at (195.6, 72.4)
- added P3: CONN_01X02, Pin_Headers:Pin_Header_Straight_1x02, F.Cu at (190.5, 90.2)
- added Q1: Q_NPN_EBC, Housings_TO-92:TO-92_Molded_Narrow, F.Cu at (172.7, 86.4)
- added R1: R, Resistors_SMD:R_0805_HandSoldering, F.Cu at (165.1, 80.0)
- added R2: R, Resistors_SMD:R_0805_HandSoldering, F.Cu at (163.8, 90.2)
- added R3: 0Ω, Resistors_SMD:R_0805_HandSoldering, F.Cu at (167.6, 85.1)
- added R4: R, Resistors_SMD:R_0805_HandSoldering, F.Cu at (172.7, 72.4)
- added R5: 0Ω, Resistors_SMD:R_0805_HandSoldering, F.Cu at (172.7, 77.5)
- added R6: 0Ω, Resistors_SMD:R_0805_HandSoldering, F.Cu at (172.7, 92.7)
- added R7: R, Resistors_SMD:R_0805_HandSoldering, F.Cu at (172.7, 97.8)

Commit message: Finalised the layout and created the Gerbers
Parts:
- added REF**: MountingHole_2-5mm, Mounting_Holes:MountingHole_2-5mm, F.Cu at (174.0, 122.2)
- added REF**: MountingHole_2-5mm, Mounting_Holes:MountingHole_2-5mm, F.Cu at (148.1, 98.6)
- added TP1: CONN_01X01, Pin_Headers:Pin_Header_Straight_1x01, F.Cu at (147.8, 106.7)
- added TP2: CONN_01X01, Pin_Headers:Pin_Header_Straight_1x01, F.Cu at (174.2, 100.1)
- moved P2 50.7 mm to (172.1, 117.3), turned to 90 degrees
- moved C3 36.1 mm to (172.7, 111.5), turned to 0 degrees
- moved P1 31.4 mm to (150.1, 116.1)
- moved R4 28.8 mm to (161.0, 98.7), turned to 0 degrees
- moved R5 27.4 mm to (161.3, 102.4), turned to 0 degrees
- moved R7 25.2 mm to (160.5, 119.9)
- moved C1 25.2 mm to (151.8, 108.5), turned to 270 degrees
- moved C2 25.0 mm to (165.4, 120.1)
- moved R1 24.9 mm to (154.7, 102.6), turned to 0 degrees
- moved R3 24.3 mm to (157.5, 107.2), turned to 180 degrees
- moved R2 24.1 mm to (156.2, 113.0)
- moved P3 23.4 mm to (172.0, 104.4)
- moved Q1 23.3 mm to (165.4, 108.5)
- moved R6 22.9 mm to (163.3, 113.5), turned to 0 degrees
- moved C4 19.1 mm to (168.1, 99.8)
Routing:
- net Net-(C1-Pad1): track 0.00 -> 13.9 mm
- net /Input: track 0.00 -> 13.7 mm
- net /Vcc: track 0.00 -> 11.2 mm, vias 0 -> 2
- net Net-(C2-Pad1): track 0.00 -> 9.88 mm
- net Net-(C4-Pad2): track 0.00 -> 9.82 mm
- net /Out: track 0.00 -> 9.52 mm
- net /Emitter: track 0.00 -> 6.78 mm
- net /Collector: track 0.00 -> 5.53 mm
- net /Base: track 0.00 -> 5.25 mm
- added copper zone on B.Cu, net /Vcc
- added copper zone on F.Cu, net GND
Other:
- board outline added: 31.5 x 29.2 mm
- net class Default: clearance 0.2 -> 0.1524; trace_width 0.25 -> 0.1524; via_dia 0.6 -> 0.6858; via_drill 0.4 -> 0.3302
- rule trace_clearance: 0.2 -> 0.1524
- rule trace_min: 0.2 -> 0.1524
- rule via_min_drill: 0.3 -> 0.3302
- rule via_min_size: 0.4 -> 0.6858
- board text added: "Input"
- board text added: "LoudMouth Rev 2L.1"
- board text added: "Out"
- board text added: "Output"
- board text added: "Vcc"
