File: ClassD/ClassD.sch (KiCad schematic (older format))
At the start: 37 parts, among them J1 RCJ-01X, J2 RCJ-01X, P1 CONN_01X02, SW1 FSM2JSMAA, U1 AP1117E50G-13, U2 TPA2008D2

Commit message: Correction to solder mask and 24-TSSOP power Pad
Connections:
- net GND: now also C6.2; no longer C6.1, U1.4 (TAB)
- net VDD: now also C6.1, U1.4 (TAB); no longer C6.2
Changed lines of the file:
@@
 	8700 3800 8800 3800
-Wire Wire Line
-	2600 1250 2600 1500
 Wire Wire Line
 	2450 1250 2450 1750
@@
 	1550 1600 2450 1600
 Connection ~ 2450 1600
-Connection ~ 2600 1500
 Text Label 4000 1050 2    60   ~ 0
 VDD
@@
 F 9 "Value" H 4150 4800 60  0001 C CNN "Fieldname"
 	1    4150 4800
-	1    0    0    -1
+	-1   0    0    1
 $EndComp
 $Comp
@@
 Text Label 5250 6300 1    60   ~ 0
 AGND
+Wire Wire Line
+	2600 1250 2600 1350
+Wire Wire Line
+	2600 1350 2950 1350
+Wire Wire Line
+	2950 1350 2950 1050
+Connection ~ 2950 1050
 $EndSCHEMATC
