File: ClassD/ClassD.kicad_pcb (KiCad board)
At the start: 2 copper layers, 64.6 x 45.3 mm, 263 parts, among them J1 RCJ-01X, J2 RCJ-01X, P1 CONN_01X02, SW1 FSM2JSMAA, U1 AP1117E50G-13, U2 TPA2008D2

Commit message: Correction to solder mask and 24-TSSOP power Pad
Parts:
- removed ST**1111161, ST**1111175: Stitch_VIA, LoudMouth-ClassD:Stitch_VIA
- turned C6 to 90 degrees
Connections:
- C6 pad 1: GND -> /VDD
- C6 pad 2: /VDD -> GND
- U1 pad 4: GND -> /VDD
Routing:
- net /VDD: track 145.3 -> 151.9 mm
Other:
- rule pad_to_mask_clearance: 0.2 -> 0
- board text added: "Loud Mouth - Class D Rev 2L_2"
- board text removed: "Loud Mouth - Class D Rev 2L_1"
Changed lines of the file:
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@@
 (kicad_pcb (version 4) (host pcbnew 4.0.2-4+6225~38~ubuntu14.04.1-stable)
   (general
-    (links 320)
+    (links 318)
     (no_connects 0)
     (area 93.284099 73.690099 167.422163 131.4834)
     (thickness 1.6)
     (drawings 15)
-    (tracks 213)
+    (tracks 214)
     (zones 0)
-    (modules 263)
+    (modules 261)
     (nets 29)
   )
   (page A4)
+  (title_block
+    (title "Load Mouth Class D")
+    (rev 2L_2)
+  )
   (layers
     (0 F.Cu signal)
@@
     (pad_size 0.6858 0.6858)
     (pad_drill 0.3302)
-    (pad_to_mask_clearance 0.2)
+    (pad_to_mask_clearance 0)
     (pad_to_paste_clearance 0.0254)
     (aux_axis_origin 0 0)
@@
   )
   (module LoudMouth-ClassD:Stitch_VIA (layer F.Cu)
-    (at 115.57 93.98)
-    (fp_text reference ST**1111175 (at 0 3.556) (layer F.SilkS) hide
-      (effects (font (size 1 1) (thickness 0.15)))
-    )
-    (fp_text value Stitch_VIA (at 0 -3.81) (layer F.Fab) hide
-      (effects (font (size 1 1) (thickness 0.15)))
-    )
-    (pad 1 thru_hole circle (at 0 0) (size 0.6858 0.6858) (drill 0.3302) (layers *.Cu)
-      (net 1 GND) (zone_connect 2))
-  )
-  (module LoudMouth-ClassD:Stitch_VIA (layer F.Cu)
     (at 113.03 93.98)
     (fp_text reference ST**1111165 (at 0 3.556) (layer F.SilkS) hide
@@
   )
   (module LoudMouth-ClassD:Stitch_VIA (layer F.Cu)
-    (at 113.03 83.82)
-    (fp_text reference ST**1111161 (at 0 3.556) (layer F.SilkS) hide
-      (effects (font (size 1 1) (thickness 0.15)))
-    )
-    (fp_text value Stitch_VIA (at 0 -3.81) (layer F.Fab) hide
-      (effects (font (size 1 1) (thickness 0.15)))
-    )
-    (pad 1 thru_hole circle (at 0 0) (size 0.6858 0.6858) (drill 0.3302) (layers *.Cu)
-      (net 1 GND) (zone_connect 2))
-  )
-  (module LoudMouth-ClassD:Stitch_VIA (layer F.Cu)
     (at 110.49 83.82)
     (fp_text reference ST**1111151 (at 0 3.556) (layer F.SilkS) hide
@@
   )
   (module Capacitors_SMD:c_elec_4x5.3 (layer F.Cu)
-    (at 124.333 86.614 270)
+    (at 124.333 86.614 90)
     (descr "SMT capacitor, aluminium electrolytic, 4x5.3")
     (attr smd)
-    (fp_text reference C6 (at 4.318 -1.905 360) (layer F.SilkS)
+    (fp_text reference C6 (at 0.889 -3.556 180) (layer F.SilkS)
       (effects (font (size 0.762 0.762) (thickness 0.127)))
     )
-    (fp_text value "10 μF" (at 0 3.175 270) (layer F.Fab)
+    (fp_text value "10 μF" (at 0 3.175 90) (layer F.Fab)
       (effects (font (size 0.762 0.762) (thickness 0.127)))
     )
@@
     (fp_line (start -2.286 -2.286) (end -2.286 2.286) (layer F.SilkS) (width 0.15))
     (fp_circle (center 0 0) (end -2.032 0) (layer F.SilkS) (width 0.15))
-    (pad 1 smd rect (at 1.80086 0 270) (size 2.60096 1.6002) (layers F.Cu F.Paste F.Mask)
-      (net 1 GND))
-    (pad 2 smd rect (at -1.80086 0 270) (size 2.60096 1.6002) (layers F.Cu F.Paste F.Mask)
+    (pad 1 smd rect (at 1.80086 0 90) (size 2.60096 1.6002) (layers F.Cu F.Paste F.Mask)
       (net 3 /VDD))
+    (pad 2 smd rect (at -1.80086 0 90) (size 2.60096 1.6002) (layers F.Cu F.Paste F.Mask)
+      (net 1 GND))
     (model Capacitors_SMD.3dshapes/c_elec_4x5.3.wrl
       (at (xyz 0 0 0))
@@
     (fp_line (start 3.556 -2.286) (end 3.556 -1.524) (layer F.SilkS) (width 0.15))
     (pad 4 smd rect (at 0 -3.302 180) (size 3.6576 2.032) (layers F.Cu F.Paste F.Mask)
-      (net 1 GND))
+      (net 3 /VDD))
     (pad 2 smd rect (at 0 3.302 180) (size 1.016 2.032) (layers F.Cu F.Paste F.Mask)
       (net 3 /VDD))
@@
       (net 10 "Net-(C13-Pad1)"))
     (pad 25 smd rect (at 0 0) (size 7.8 3.4) (layers F.Cu F.Paste F.Mask)
-      (net 1 GND) (solder_mask_margin -0.2) (zone_connect 2))
+      (net 1 GND) (solder_paste_margin -0.5) (zone_connect 2))
     (pad 25 smd rect (at 0 0) (size 7.8 3.4) (layers B.Cu)
       (net 1 GND) (solder_mask_margin 1) (zone_connect 2))
@@
     (effects (font (size 1.5 1.5) (thickness 0.3)) (justify left))
   )
-  (gr_text "Loud Mouth - Class D\nRev 2L_1" (at 120.904 106.299) (layer F.SilkS)
+  (gr_text "Loud Mouth - Class D\nRev 2L_2" (at 120.904 106.299) (layer F.SilkS)
     (effects (font (size 1.016 1.016) (thickness 0.127)) (justify left))
   )
@@
   (segment (start 112.969 87.503) (end 112.776 87.696) (width 1.2192) (layer F.Cu) (net 2))
   (segment (start 112.776 87.696) (end 112.776 90.424) (width 1.2192) (layer F.Cu) (net 2))
+  (segment (start 124.333 84.81314) (end 125.19914 83.947) (width 1.2192) (layer F.Cu) (net 3))
+  (segment (start 125.19914 83.947) (end 135.382 83.947) (width 1.2192) (layer F.Cu) (net 3))
+  (segment (start 122.15114 86.995) (end 124.333 84.81314) (width 1.2192) (layer F.Cu) (net 3))
+  (segment (start 115.062 97.028) (end 115.062 90.424) (width 0.6096) (layer F.Cu) (net 3))
   (segment (start 147.066 100.33) (end 147.193 100.33) (width 0.6096) (layer B.Cu) (net 3))
   (segment (start 147.193 100.33) (end 148.844 98.679) (width 0.6096) (layer B.Cu) (net 3))
@@
   (segment (start 158.623 104.648) (end 158.623 109.855) (width 0.6096) (layer F.Cu) (net 3))
   (segment (start 156.956 102.981) (end 158.623 104.648) (width 0.6096) (layer F.Cu) (net 3))
-  (segment (start 124.333 84.81314) (end 125.19914 83.947) (width 1.2192) (layer F.Cu) (net 3))
   (segment (start 136.358 84.923) (end 136.358 86.106) (width 1.2192) (layer F.Cu) (net 3))
   (segment (start 135.382 83.947) (end 136.358 84.923) (width 1.2192) (layer F.Cu) (net 3))
-  (segment (start 125.19914 83.947) (end 135.382 83.947) (width 1.2192) (layer F.Cu) (net 3))
   (segment (start 115.062 90.424) (end 115.062 89.662) (width 1.2192) (layer F.Cu) (net 3))
   (segment (start 115.062 89.662) (end 117.729 86.995) (width 1.2192) (layer F.Cu) (net 3))
-  (segment (start 122.15114 86.995) (end 124.333 84.81314) (width 1.2192) (layer F.Cu) (net 3))
   (segment (start 117.729 86.995) (end 122.15114 86.995) (width 1.2192) (layer F.Cu) (net 3))
   (segment (start 115.062 90.424) (end 115.062 87.696) (width 0.6096) (layer F.Cu) (net 3))
